File: hardware/cda-pcb/cda-pcb.kicad_pcb (KiCad board)
At the start: 4 copper layers, 112 x 127 mm, 202 parts, among them J1 ICD15S13E4GX00LF, J2 ICD15S13E4GX00LF, J3 ICD15S13E4GX00LF, J4 ICD15S13E4GX00LF, J5 Conn_01x06, P1 0022272021, U1 ADS124S08IRHBT, U10 SN74AHCT125RGYR, U2 ADS124S08IRHBT, U3 ADS124S08IRHBT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

Commit message: lowk idr if I changed anything
Routing:
- net GND: track 111.1 -> 137.8 mm, vias 90 -> 89
- net +6V: track 73.6 -> 77.3 mm
- net (no net): track 2.92 -> 0.00 mm
- net +11V: track 50.6 -> 52.6 mm
Other:
- board text removed: "U3"

Commit message: addfed stitching vias
Modify PCB to add numerous free vias (mostly on net 2/GND) and refresh UUIDs for multiple pads/power pins. Updated cda-pcb.kicad_pcb with many new via entries and coordinate adjustments; supporting KiCad files (cda-pcb.kicad_prl, cda-pcb.kicad_sch, fp-info-cache) were also updated. Several old backup ZIPs under hardware/cda-pcb/cda-pcb-backups were removed and new timestamped backups were added.
Routing:
- net GND: vias 89 -> 336

Commit message: changed 10Vs buck output to be 9.988V and added a 2nd 10Vs dsub pin
Parts:
- R25: value 24k -> 13k
- R26: value 3.3k -> 1.8k
- moved G*** 29.0 mm to (113.6, 150.9)
- moved G*** 5.86 mm to (81.4, 150.5)
- moved G*** 4.67 mm to (96.7, 150.9)
Connections:
- J3 pad 15: +5Vs -> +10Vs
Routing:
- net +10Vs: track 104.9 -> 152.7 mm
- net +5Vs: track 479.8 -> 513.4 mm, vias 14 -> 13
- net GND: vias 336 -> 88
